File: hardware/BioAmp-EMG-Pill.sch (KiCad schematic (older format))
At the start: 27 parts, among them J1 Conn_01x03, J3 Conn_01x04, U1 TL074

Commit message: Update to v0.5
Tested circuit, working great!
Parts:
- removed C5, C6: 10uf, Capacitor_SMD:C_0805_2012Metric_Pad1.18x1.45mm_HandSolder, symbol Device:C
- removed D2: D, Diode_SMD:D_0805_2012Metric_Pad1.15x1.40mm_HandSolder, symbol Device:D
- removed H1: MountingHole_Pad, MountingHole:MountingHole_2.5mm_Pad_Via, symbol Mechanical:MountingHole_Pad
- removed J3: Conn_01x04, Connector_PinSocket_2.54mm:PinSocket_1x04_P2.54mm_Vertical, symbol Connector_Generic:Conn_01x04
- removed R12: 10k, Resistor_SMD:R_0805_2012Metric_Pad1.20x1.40mm_HandSolder, symbol Device:R
- added D2: LED, LED_SMD:LED_0603_1608Metric_Castellated, symbol Device:LED
- added J2: Conn_01x03, Connector_PinHeader_2.54mm:PinHeader_1x03_P2.54mm_Vertical, symbol Connector_Generic:Conn_01x03
- C1: value 1uf -> 2.2uf; footprint Capacitor_SMD:C_0805_2012Metric_Pad1.18x1.45mm_HandSolder -> Capacitor_SMD:C_0603_1608Metric_Pad1.08x0.95mm_HandSolder
- C2: value 1.5nf -> 100pf; footprint Capacitor_SMD:C_0805_2012Metric_Pad1.18x1.45mm_HandSolder -> Capacitor_SMD:C_0603_1608Metric_Pad1.08x0.95mm_HandSolder
- C3, C4: value 10uf -> 100n; footprint Capacitor_SMD:C_0805_2012Metric_Pad1.18x1.45mm_HandSolder -> Capacitor_SMD:C_0603_1608Metric_Pad1.08x0.95mm_HandSolder
- C7, C8, C9: footprint Capacitor_SMD:C_0805_2012Metric_Pad1.18x1.45mm_HandSolder -> Capacitor_SMD:C_0603_1608Metric_Pad1.08x0.95mm_HandSolder
- J1: footprint Connector_JST:JST_EH_S3B-EH_1x03_P2.50mm_Horizontal -> Connector_PinHeader_2.54mm:PinHeader_1x03_P2.54mm_Vertical
- R1, R2, R3, R4, R5, R6, R8, R9: footprint Resistor_SMD:R_0805_2012Metric_Pad1.20x1.40mm_HandSolder -> Resistor_SMD:R_0603_1608Metric_Pad0.98x0.95mm_HandSolder
- R10: value 1k -> 1M; footprint Resistor_SMD:R_0805_2012Metric_Pad1.20x1.40mm_HandSolder -> Resistor_SMD:R_0603_1608Metric_Pad0.98x0.95mm_HandSolder
- R11: value 100k -> 1k; footprint Resistor_SMD:R_0805_2012Metric_Pad1.20x1.40mm_HandSolder -> Resistor_SMD:R_0603_1608Metric_Pad0.98x0.95mm_HandSolder
- R7: value 100k -> 1M; footprint Resistor_SMD:R_0805_2012Metric_Pad1.20x1.40mm_HandSolder -> Resistor_SMD:R_0603_1608Metric_Pad0.98x0.95mm_HandSolder
Connections:
- net AMP2 is gone; now on net OUT: C2.1, R7.1, U1.8
- net GND: now also R11.1, J2.2 (Pin_2); no longer J1.1 (Pin_1), U1.12 (+)
- net OUT: now also D2.2 (A), J2.1 (Pin_1)
- net VCC: now also J2.3 (Pin_3)
- net vRef: now also U1.12 (+)
- net DRLin: now reaches R2.1, R3.2, U1.1
- net DRLin: now also R10.2, U1.13 (-)
- net DRL: now reaches R10.1
- net DRL: now also J1.1 (Pin_1), U1.14
- net RAW: no longer names the net of R11.2
- net RAW: now also D2.1 (K); no longer U1.14
Other:
- note added: "1000x Gain (Bandpass 75Hz - 2000Hz)"
- note added: "Driven right leg"
- note removed: "100x Gain"
- note removed: "100x Gain (Bandpass 150Hz - 1050Hz)"
- moved on the sheet: C1, C2, D1, J1, R5, R6, R7, U1C, U1D

Commit message: Update to v0.6
Parts:
- removed D1, D2: LED, LED_SMD:LED_0603_1608Metric_Castellated, symbol Device:LED
- added C5: 1nf, Capacitor_SMD:C_0603_1608Metric_Pad1.08x0.95mm_HandSolder, symbol Device:C
- added R12: 100k, Resistor_SMD:R_0603_1608Metric_Pad0.98x0.95mm_HandSolder, symbol Device:R
- C8: value 10uf -> 2.2uf
- R11, R6: value 1k -> 100k
Connections:
- net BIO+: now also R12.2; no longer U1.5 (+)
- net BIO-: now also R6.2; no longer U1.3 (+)
- net DRL: now also R11.1; no longer R10.1, U1.14
- net DRLin: now also C5.1
- net GND: no longer R11.1, R6.1
- net at R11.2: now also R10.1, U1.14, C5.2
- new net: R6.1, U1.3 (+)
- new net: R12.1, U1.5 (+)
Other:
- moved on the sheet: C1, C2, C9, J1, J2, R1, R10, R2, R3, R4, R5, R7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

Commit message: update PCB
Parts:
- C1: value 2.2uf -> 47uf; footprint Capacitor_SMD:C_0603_1608Metric_Pad1.08x0.95mm_HandSolder -> Capacitor_SMD:C_0805_2012Metric_Pad1.18x1.45mm_HandSolder
Other:
- moved on the sheet: C3, C4, C7, C8, R8, R9
Changed lines of the file:
@@
 P 3370 4155
 F 0 "C1" V 3118 4155 50  0000 C CNN
-F 1 "2.2uf" V 3209 4155 50  0000 C CNN
-F 2 "Capacitor_SMD:C_0603_1608Metric_Pad1.08x0.95mm_HandSolder" H 3408 4005 50  0001 C CNN
+F 1 "47uf" V 3209 4155 50  0000 C CNN
+F 2 "Capacitor_SMD:C_0805_2012Metric_Pad1.18x1.45mm_HandSolder" H 3408 4005 50  0001 C CNN
 F 3 "~" H 3370 4155 50  0001 C CNN
 	1    3370 4155
@@
 L Device:R R8
 U 1 1 6035DAA0
-P 8305 990
-F 0 "R8" H 8255 1005 50  0000 R CNN
-F 1 "10k" V 8300 1055 50  0000 R CNN
-F 2 "Resistor_SMD:R_0603_1608Metric_Pad0.98x0.95mm_HandSolder" V 8235 990 50  0001 C CNN
-F 3 "~" H 8305 990 50  0001 C CNN
-	1    8305 990
+P 8220 1185
+F 0 "R8" H 8170 1200 50  0000 R CNN
+F 1 "10k" V 8215 1250 50  0000 R CNN
+F 2 "Resistor_SMD:R_0603_1608Metric_Pad0.98x0.95mm_HandSolder" V 8150 1185 50  0001 C CNN
+F 3 "~" H 8220 1185 50  0001 C CNN
+	1    8220 1185
 	-1   0    0    1
 $EndComp
@@
 L Device:R R9
 U 1 1 6036797A
-P 8305 1290
-F 0 "R9" H 8250 1290 50  0000 R CNN
-F 1 "10k" V 8300 1360 50  0000 R CNN
-F 2 "Resistor_SMD:R_0603_1608Metric_Pad0.98x0.95mm_HandSolder" V 8235 1290 50  0001 C CNN
-F 3 "~" H 8305 1290 50  0001 C CNN
-	1    8305 1290
+P 8220 1485
+F 0 "R9" H 8165 1485 50  0000 R CNN
+F 1 "10k" V 8215 1555 50  0000 R CNN
+F 2 "Resistor_SMD:R_0603_1608Metric_Pad0.98x0.95mm_HandSolder" V 8150 1485 50  0001 C CNN
+F 3 "~" H 8220 1485 50  0001 C CNN
+	1    8220 1485
 	-1   0    0    1
 $EndComp
 Wire Wire Line
-	7955 840  8155 840
-Wire Wire Line
-	7955 1440 8155 1440
-Wire Wire Line
-	7955 1140 8305 1140
-Connection ~ 8305 1140
+	7870 1035 8070 1035
+Wire Wire Line
+	7870 1635 8070 1635
+Wire Wire Line
+	7870 1335 8220 1335
+Connection ~ 8220 1335
 $Comp
 L power:VCC #PWR0107
 U 1 1 60378EF6
-P 8155 840
-F 0 "#PWR0107" H 8155 690 50  0001 C CNN
-F 1 "VCC" H 8170 1013 50  0000 C CNN
-F 2 "" H 8155 840 50  0001 C CNN
-F 3 "" H 8155 840 50  0001 C CNN
-	1    8155 840
-	1    0    0    -1
-$EndComp
-Connection ~ 8155 840
-Wire Wire Line
-	8155 840  8305 840
+P 8070 1035
+F 0 "#PWR0107" H 8070 885 50  0001 C CNN
+F 1 "VCC" H 8085 1208 50  0000 C CNN
+F 2 "" H 8070 1035 50  0001 C CNN
+F 3 "" H 8070 1035 50  0001 C CNN
+	1    8070 1035
+	1    0    0    -1
+$EndComp
+Connection ~ 8070 1035
+Wire Wire Line
+	8070 1035 8220 1035
 $Comp
 L power:GND #PWR0108
 U 1 1 603795E1
-P 8155 1440
-F 0 "#PWR0108" H 8155 1190 50  0001 C CNN
-F 1 "GND" H 8160 1267 50  0000 C CNN
-F 2 "" H 8155 1440 50  0001 C CNN
-F 3 "" H 8155 1440 50  0001 C CNN
-	1    8155 1440
-	1    0    0    -1
-$EndComp
-Connection ~ 8155 1440
-Wire Wire Line
-	8155 1440 8305 1440
-Text GLabel 8555 1140 2    50   Input ~ 0
+P 8070 1635
+F 0 "#PWR0108" H 8070 1385 50  0001 C CNN
+F 1 "GND" H 8075 1462 50  0000 C CNN
+F 2 "" H 8070 1635 50  0001 C CNN
+F 3 "" H 8070 1635 50  0001 C CNN
+	1    8070 1635
+	1    0    0    -1
+$EndComp
+Connection ~ 8070 1635
+Wire Wire Line
+	8070 1635 8220 1635
+Text GLabel 8470 1335 2    50   Input ~ 0
 vRef
 Wire Wire Line
-	8305 1140 8555 1140
+	8220 1335 8470 1335
 $Comp
 L Device:C C3
 U 1 1 603F1D18
-P 7955 990
-F 0 "C3" V 7705 990 50  0000 C CNN
-F 1 "100n" V 7805 990 50  0000 C CNN
-F 2 "Capacitor_SMD:C_0603_1608Metric_Pad1.08x0.95mm_HandSolder" H 7993 840 50  0001 C CNN
-F 3 "~" H 7955 990 50  0001 C CNN
-	1    7955 990
+P 7870 1185
+F 0 "C3" V 7620 1185 50  0000 C CNN
+F 1 "100n" V 7720 1185 50  0000 C CNN
+F 2 "Capacitor_SMD:C_0603_1608Metric_Pad1.08x0.95mm_HandSolder" H 7908 1035 50  0001 C CNN
+F 3 "~" H 7870 1185 50  0001 C CNN
+	1    7870 1185
 	1    0    0    -1
 $EndComp
@@
 L Device:C C4
 U 1 1 603F6543
-P 7955 1290
-F 0 "C4" V 7705 1290 50  0000 C CNN
-F 1 "100n" V 7805 1290 50  0000 C CNN
-F 2 "Capacitor_SMD:C_0603_1608Metric_Pad1.08x0.95mm_HandSolder" H 7993 1140 50  0001 C CNN
-F 3 "~" H 7955 1290 50  0001 C CNN
-	1    7955 1290
-	1    0    0    -1
-$EndComp
-Connection ~ 7955 1140
+P 7870 1485
+F 0 "C4" V 7620 1485 50  0000 C CNN
+F 1 "100n" V 7720 1485 50  0000 C CNN
+F 2 "Capacitor_SMD:C_0603_1608Metric_Pad1.08x0.95mm_HandSolder" H 7908 1335 50  0001 C CNN
+F 3 "~" H 7870 1485 50  0001 C CNN
+	1    7870 1485
+	1    0    0    -1
+$EndComp
+Connection ~ 7870 1335
 $Comp
 L Connector_Generic:Conn_01x03 J1
@@
 L Device:C C7
 U 1 1 60682C1F
-P 10000 1150
-F 0 "C7" V 9750 1150 50  0000 C CNN
-F 1 "100nf" V 9850 1150 50  0000 C CNN
-F 2 "Capacitor_SMD:C_0603_1608Metric_Pad1.08x0.95mm_HandSolder" H 10038 1000 50  0001 C CNN
-F 3 "~" H 10000 1150 50  0001 C CNN
-	1    10000 1150
+P 10000 1320
+F 0 "C7" V 9750 1320 50  0000 C CNN
+F 1 "100nf" V 9850 1320 50  0000 C CNN
+F 2 "Capacitor_SMD:C_0603_1608Metric_Pad1.08x0.95mm_HandSolder" H 10038 1170 50  0001 C CNN
+F 3 "~" H 10000 1320 50  0001 C CNN
+	1    10000 1320
 	1    0    0    -1
 $EndComp
@@
 L power:VCC #PWR0102
 U 1 1 606933C3
-P 10200 1000
-F 0 "#PWR0102" H 10200 850 50  0001 C CNN
-F 1 "VCC" H 10215 1173 50  0000 C CNN
-F 2 "" H 10200 1000 50  0001 C CNN
-F 3 "" H 10200 1000 50  0001 C CNN
-	1    10200 1000
+P 10200 1170
+F 0 "#PWR0102" H 10200 1020 50  0001 C CNN
+F 1 "VCC" H 10215 1343 50  0000 C CNN
+F 2 "" H 10200 1170 50  0001 C CNN
+F 3 "" H 10200 1170 50  0001 C CNN
+	1    10200 1170
 	1    0    0    -1
 $EndComp
@@
 L power:GND #PWR0113
 U 1 1 6069403E
-P 10200 1300
-F 0 "#PWR0113" H 10200 1050 50  0001 C CNN
-F 1 "GND" H 10205 1127 50  0000 C CNN
-F 2 "" H 10200 1300 50  0001 C CNN
-F 3 "" H 10200 1300 50  0001 C CNN
-	1    10200 1300
-	1    0    0    -1
-$EndComp
-Wire Wire Line
-	10000 1000 10200 1000
-Connection ~ 10200 1000
-Wire Wire Line
-	10200 1000 10400 1000
-Wire Wire Line
-	10000 1300 10200 1300
-Connection ~ 10200 1300
-Wire Wire Line
-	10200 1300 10400 1300
+P 10200 1470
+F 0 "#PWR0113" H 10200 1220 50  0001 C CNN
+F 1 "GND" H 10205 1297 50  0000 C CNN
+F 2 "" H 10200 1470 50  0001 C CNN
+F 3 "" H 10200 1470 50  0001 C CNN
+	1    10200 1470
+	1    0    0    -1
+$EndComp
+Wire Wire Line
+	10000 1170 10200 1170
+Connection ~ 10200 1170
+Wire Wire Line
+	10200 1170 10400 1170
+Wire Wire Line
+	10000 1470 10200 1470
+Connection ~ 10200 1470
+Wire Wire Line
+	10200 1470 10400 1470
 Text Notes 2900 2700 0    79   ~ 0
 10x Gain Instrumentation Amp
@@
 L Device:C C8
 U 1 1 601A5E02
-P 10400 1150
-F 0 "C8" V 10150 1150 50  0000 C CNN
-F 1 "2.2uf" V 10250 1150 50  0000 C CNN
-F 2 "Capacitor_SMD:C_0603_1608Metric_Pad1.08x0.95mm_HandSolder" H 10438 1000 50  0001 C CNN
-F 3 "~" H 10400 1150 50  0001 C CNN
-	1    10400 1150
+P 10400 1320
+F 0 "C8" V 10150 1320 50  0000 C CNN
+F 1 "2.2uf" V 10250 1320 50  0000 C CNN
+F 2 "Capacitor_SMD:C_0603_1608Metric_Pad1.08x0.95mm_HandSolder" H 10438 1170 50  0001 C CNN
+F 3 "~" H 10400 1320 50  0001 C CNN
+	1    10400 1320
 	-1   0    0    1
 $EndComp
